Commit message: changed robot design

File: my_robot/urdf/my_robot.xacro (robot description, xacro)
@@ -12,5 +12,5 @@
     <inertial>
       <mass value="15.0"/>
-      <origin xyz="0.1 0 0" rpy=" 0 0 0"/>
+      <origin xyz="0.0 0 0" rpy=" 0 0 0"/>
       <inertia
           ixx="0.1" ixy="0" ixz="0"
@@ -22,5 +22,5 @@
       <origin xyz="0 0 0" rpy=" 0 0 0"/>
       <geometry>
-        <cylinder radius=".25" length=".2"/>
+        <cylinder radius=".15" length=".1"/>
       </geometry>
     </collision>
@@ -28,5 +28,5 @@
       <origin xyz="0 0 0" rpy=" 0 0 0"/>
       <geometry>
-        <cylinder radius=".25" length=".2"/>
+        <cylinder radius=".15" length=".1"/>
       </geometry>
       <material name="Blue">
@@ -35,5 +35,5 @@
     </visual>
     <collision name='front_caster_collision'>
-      <origin xyz="0.2 0 -0.1" rpy=" 0 0 0"/>
+      <origin xyz="0.1 0 -0.025" rpy=" 0 0 0"/>
       <geometry>
         <sphere radius="0.0499"/>
@@ -41,5 +41,5 @@
     </collision>
     <visual name='front_caster_visual'>
-      <origin xyz="0.2 0 -0.1" rpy=" 0 0 0"/>
+      <origin xyz="0.1 0 -0.025" rpy=" 0 0 0"/>
       <geometry>
         <sphere radius="0.05"/>
@@ -50,5 +50,5 @@
    </visual>
     <collision name='rear_caster_collision'>
-      <origin xyz="-0.2 0 -0.1" rpy=" 0 0 0"/>
+      <origin xyz="-0.1 0 -0.025" rpy=" 0 0 0"/>
       <geometry>
         <sphere radius="0.0499"/>
@@ -56,5 +56,5 @@
     </collision>
     <visual name='rear_caster_visual'>
-      <origin xyz="-0.2 0 -0.1" rpy=" 0 0 0"/>
+      <origin xyz="-0.1 0 -0.025" rpy=" 0 0 0"/>
       <geometry>
         <sphere radius="0.05"/>
@@ -79,8 +79,8 @@
       />
     </inertial>
-    <collision name='collision'>
+    <collision name='left_wheel_collision'>
       <origin xyz="0 0 0" rpy=" 0 1.57 1.57"/>
       <geometry>
-        <cylinder radius=".125" length="0.05"/>
+        <cylinder radius=".05" length="0.025"/>
       </geometry>
     </collision>
@@ -88,5 +88,5 @@
       <origin xyz="0 0 0" rpy=" 0 1.57 1.57"/>
       <geometry>
-        <cylinder radius=".125" length="0.05"/>
+        <cylinder radius=".05" length="0.025"/>
       </geometry>
     </visual>
@@ -103,19 +103,19 @@
       />
     </inertial>
-    <collision name='collision'>
+    <collision name='right_wheel_collision'>
       <origin xyz="0 0 0" rpy=" 0 1.57 1.57"/>
       <geometry>
-        <cylinder radius=".125" length="0.05"/>
+        <cylinder radius=".05" length="0.025"/>
       </geometry>
     </collision>
-    <visual name='left_wheel_visual'>
+    <visual name='right_wheel_visual'>
       <origin xyz="0 0 0" rpy=" 0 1.57 1.57"/>
       <geometry>
-        <cylinder radius=".125" length="0.05"/>
+        <cylinder radius=".05" length="0.025"/>
       </geometry>
     </visual>
   </link>
  <joint type="continuous" name="left_wheel_hinge">
-    <origin xyz="0 0.275 -0.025" rpy="0 0 0"/>
+    <origin xyz="0 0.125 -0.025" rpy="0 0 0"/>
     <child link="left_wheel"/>
     <parent link="chassis"/>
@@ -125,5 +125,5 @@
   </joint>
  <joint type="continuous" name="right_wheel_hinge">
-    <origin xyz="0 -0.275 -0.025" rpy="0 0 0"/>
+    <origin xyz="0 -0.125 -0.025" rpy="0 0 0"/>
     <child link="right_wheel"/>
     <parent link="chassis"/>
@@ -143,5 +143,5 @@
       />
     </inertial>
-    <collision name='collision'>
+    <collision name='camera_collision'>
       <origin xyz="0 0 0" rpy=" 0 0 0"/>
       <geometry>
@@ -149,5 +149,5 @@
       </geometry>
     </collision>
-    <visual name='left_wheel_visual'>
+    <visual name='camera_visual'>
       <origin xyz="0 0 0" rpy=" 0 0 0"/>
       <geometry>
@@ -157,5 +157,5 @@
   </link>
  <joint type="fixed" name="camera_joint">
-    <origin xyz="0.25 0 0.0" rpy="0 0 0"/>
+    <origin xyz="0.15 0 0.0" rpy="0 0 0"/>
     <child link="camera"/>
     <parent link="chassis"/>
@@ -173,5 +173,5 @@
       />
     </inertial>
-    <collision name='collision'>
+    <collision name='hokuyo_collision'>
       <origin xyz="0 0 0" rpy=" 0 0 0"/>
       <geometry>
@@ -179,5 +179,5 @@
       </geometry>
     </collision>
-    <visual name='left_wheel_visual'>
+    <visual name='hokuyo_visual'>
       <origin xyz="0 0 0" rpy=" 0 0 0"/>
       <geometry>
@@ -187,5 +187,5 @@
   </link>
  <joint type="fixed" name="hokuyo_joint">
-    <origin xyz="0 0 0.125" rpy="0 0 0"/>
+    <origin xyz="0 0 0.075" rpy="0 0 0"/>
     <child link="hokuyo"/>
     <parent link="chassis"/>

Commit message: configured RTAB-map and updated documentation

File: my_robot/urdf/my_robot.xacro (robot description, xacro)
@@ -132,5 +132,5 @@
     <dynamics damping="1.0" friction="1.0"/>
   </joint>
-  <link name='camera'>
+  <link name='camera_link'>
     <pose>0 0 0 0 0 0</pose>
     <inertial>
@@ -157,6 +157,6 @@
   </link>
  <joint type="fixed" name="camera_joint">
-    <origin xyz="0.15 0 0.0" rpy="0 0 0"/>
-    <child link="camera"/>
+    <origin xyz="0.15 0 0.0" rpy="0 -0.1 0"/>
+    <child link="camera_link"/>
     <parent link="chassis"/>
     <axis xyz="0 1 0" rpy="0 0 0"/>
@@ -192,6 +192,13 @@
     <axis xyz="0 1 0" rpy="0 0 0"/>
   </joint>
-<gazebo reference="camera">
+<gazebo reference="camera_link">
     <material>Gazebo/Red</material>
 </gazebo>
+  <joint name="camera_optical_joint" type="fixed">
+    <origin xyz="0 0 0" rpy="-1.5707 0 -1.5707"/>
+    <parent link="camera_link"/>
+    <child link="camera_link_optical"/>
+  </joint>
+  <link name="camera_link_optical">
+  </link>
 </robot>
